Commit message: built model prototype, cup spawning

File: src/model/urdf/model.urdf (robot description, URDF)
Before this commit: robot firefighter, 1 links, 0 joints
Links:
- added link bolt; visual cylinder length=${bolt['l']} radius=${bolt['r']}
- added link leg; visual box size=${leg['x']} ${leg['y']} ${leg['z']}
- added link nozzle; visual cylinder length=${nozzle['l']} radius=${nozzle['r']}
- added link servo; visual box size=${servo['x']} ${servo['y']} ${servo['z']}
- added link wheel; visual cylinder length=${wheel['l']} radius=${wheel['r']}
- link base_link: geometry visual box size=${servo['x']} ${servo['y']} ${servo['z']}
Joints:
- added joint bolt_to_leg: type fixed, parent bolt, child leg, origin xyz=${bolt['l']-leg['x']/2} 0 0
- added joint bolt_to_nozzle: type prismatic, parent bolt, child nozzle, origin xyz=0 0 0, limit lower=${nozzle['l']/2} upper=${bolt['l']-nozzle['l']/2-leg['x']} effort=250.0 velocity=0.5
- added joint j1: type revolute, parent base_link, child servo, origin xyz=0 0 ${servo['z']/2}, axis 0.0 0.0 1, limit lower=-3.14 upper=3.14 effort=250.0 velocity=0.5
- added joint leg_to_wheel: type fixed, parent leg, child wheel, origin xyz=0 0 ${-leg['z']}
- added joint servo_to_bolt: type fixed, parent servo, child bolt, origin xyz=${servo['x']/2} 0 ${servo['z']/2}

Commit message: colors fixed launch, fixed cup_publisher name

File: src/model/urdf/model.urdf (robot description, URDF)
Before this commit: robot firefighter, 6 links, 5 joints
Joints:
- joint leg_to_wheel: origin xyz=0 0 ${-leg['z']} -> xyz=${(leg['x']+wheel['l'])/2} 0 ${-leg['z']}
